File: gb-cart-arduino-v2/gb-cart-arduino-v2.kicad_sch (KiCad schematic)
At the start: 18 parts, among them J1 Conn_01x16_Pin, U1 74HC595, U2 74HC595

Commit message: Rewired v2
Parts:
- renumbered Ce1 to C1, Rd8 to Rd0, Rd7 to Rd1, Rd6 to Rd2, Rd5 to Rd3, Rd3 to Rd5, Rd2 to Rd6, Rd1 to Rd7, Ra4 to Rl1, Ra2 to Rr1, Ra1 to Rw1
Connections:
- net Address_Clock: now also J1.8 (Pin_8); no longer J1.7 (Pin_7)
- net Address_Latch: now also J1.7 (Pin_7); no longer J1.8 (Pin_8)
- net VCC: no longer D1.2 (A), Rl1.1
- new net LED: D1.2 (A), Rl1.1
Changed lines of the file:
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@@
 	)
 	(junction
+		(at 187.96 30.48)
+		(diameter 0)
+		(color 0 0 0 0)
+	)
+	(junction
 		(at 177.8 30.48)
 		(diameter 0)
@@
 	(wire
 		(pts
-			(xy 78.74 97.79) (xy 36.83 97.79)
-		)
-		(stroke
-			(width 0)
-			(type default)
-		)
-	)
-	(wire
-		(pts
 			(xy 143.51 107.95) (xy 143.51 97.79)
 		)
@@
 	(wire
 		(pts
+			(xy 187.96 30.48) (xy 189.23 30.48)
+		)
+		(stroke
+			(width 0)
+			(type default)
+		)
+	)
+	(wire
+		(pts
 			(xy 128.27 92.71) (xy 218.44 92.71)
 		)
@@
 	(wire
 		(pts
-			(xy 77.47 143.51) (xy 168.91 143.51)
+			(xy 36.83 95.25) (xy 77.47 95.25)
 		)
 		(stroke
@@
 	(wire
 		(pts
-			(xy 138.43 82.55) (xy 218.44 82.55)
+			(xy 77.47 143.51) (xy 168.91 143.51)
 		)
 		(stroke
@@
 	(wire
 		(pts
-			(xy 77.47 95.25) (xy 36.83 95.25)
+			(xy 138.43 82.55) (xy 218.44 82.55)
 		)
 		(stroke
@@
 	(wire
 		(pts
-			(xy 78.74 77.47) (xy 81.28 77.47)
+			(xy 77.47 77.47) (xy 81.28 77.47)
 		)
 		(stroke
@@
 	(wire
 		(pts
-			(xy 77.47 69.85) (xy 77.47 95.25)
+			(xy 80.01 69.85) (xy 80.01 97.79)
 		)
 		(stroke
@@
 	(wire
 		(pts
-			(xy 78.74 77.47) (xy 78.74 97.79)
+			(xy 90.17 135.89) (xy 90.17 123.19)
 		)
 		(stroke
@@
 	(wire
 		(pts
-			(xy 90.17 135.89) (xy 90.17 123.19)
+			(xy 77.47 77.47) (xy 77.47 95.25)
 		)
 		(stroke
@@
 	(wire
 		(pts
-			(xy 187.96 30.48) (xy 189.23 30.48)
-		)
-		(stroke
-			(width 0)
-			(type default)
-		)
-	)
-	(wire
-		(pts
 			(xy 83.82 72.39) (xy 102.87 72.39)
 		)
@@
 	(wire
 		(pts
-			(xy 77.47 69.85) (xy 96.52 69.85)
+			(xy 80.01 69.85) (xy 96.52 69.85)
 		)
 		(stroke
@@
 	(wire
 		(pts
+			(xy 186.69 30.48) (xy 187.96 30.48)
+		)
+		(stroke
+			(width 0)
+			(type default)
+		)
+	)
+	(wire
+		(pts
 			(xy 158.75 123.19) (xy 158.75 113.03)
 		)
@@
 	(wire
 		(pts
+			(xy 36.83 97.79) (xy 80.01 97.79)
+		)
+		(stroke
+			(width 0)
+			(type default)
+		)
+	)
+	(wire
+		(pts
 			(xy 80.01 100.33) (xy 36.83 100.33)
 		)
@@
 		)
 	)
-	(label "VCC"
-		(at 187.96 30.48 0)
+	(label "LED"
+		(at 186.69 30.48 0)
 		(effects
 			(font
@@
 	)
 	(label "Address_Clock"
-		(at 39.37 95.25 0)
+		(at 39.37 97.79 0)
 		(effects
 			(font
@@
 	)
 	(label "Address_Latch"
-		(at 39.37 97.79 0)
+		(at 39.37 95.25 0)
 		(effects
 			(font
@@
 		(dnp no)
 		(fields_autoplaced yes)
-		(property "Reference" "Ce1"
+		(property "Reference" "C1"
 			(at 184.6961 60.96 0)
 			(effects
@@
 			(project "gb-cart-arduino-v2"
 				(path "/9cf3a41e-ce13-4647-b5c2-ee25df0afcb2"
-					(reference "Ce1")
+					(reference "C1")
 					(unit 1)
 				)
@@
 		(on_board yes)
 		(dnp no)
-		(property "Reference" "Rd8"
+		(property "Reference" "Rd0"
 			(at 204.47 152.4 0)
 			(effects
@@
 			(project "gb-cart-arduino-v2"
 				(path "/9cf3a41e-ce13-4647-b5c2-ee25df0afcb2"
-					(reference "Rd8")
+					(reference "Rd0")
 					(unit 1)
 				)
@@
 		(on_board yes)
 		(dnp no)
-		(property "Reference" "Ra2"
+		(property "Reference" "Rr1"
 			(at 182.88 52.07 90)
 			(effects
@@
 			(project "gb-cart-arduino-v2"
 				(path "/9cf3a41e-ce13-4647-b5c2-ee25df0afcb2"
-					(reference "Ra2")
+					(reference "Rr1")
 					(unit 1)
 				)
@@
 		(on_board yes)
 		(dnp no)
-		(property "Reference" "Rd5"
+		(property "Reference" "Rd3"
 			(at 196.85 152.4 0)
 			(effects
@@
 			(project "gb-cart-arduino-v2"
 				(path "/9cf3a41e-ce13-4647-b5c2-ee25df0afcb2"
-					(reference "Rd5")
+					(reference "Rd3")
 					(unit 1)
 				)
@@
 		(on_board yes)
 		(dnp no)
-		(property "Reference" "Rd3"
+		(property "Reference" "Rd5"
 			(at 191.77 152.4 0)
 			(effects
@@
 			(project "gb-cart-arduino-v2"
 				(path "/9cf3a41e-ce13-4647-b5c2-ee25df0afcb2"
-					(reference "Rd3")
+					(reference "Rd5")
 					(unit 1)
 				)
@@
 		(on_board yes)
 		(dnp no)
-		(fields_autoplaced yes)
 		(property "Reference" "D1"
 			(at 182.5625 24.13 0)
@@
 		)
 		(property "Description" "Light emitting diode"
-			(at 184.15 30.48 0)
+			(at 178.562 27.686 0)
 			(effects
 				(font
 					(size 1.27 1.27)
 				)
+				(hide yes)
 			)
 		)
@@
 		(on_board yes)
 		(dnp no)
-		(property "Reference" "Rd2"
+		(property "Reference" "Rd6"
 			(at 189.23 152.4 0)
 			(effects
@@
 			(project "gb-cart-arduino-v2"
 				(path "/9cf3a41e-ce13-4647-b5c2-ee25df0afcb2"
-					(reference "Rd2")
+					(reference "Rd6")
 					(unit 1)
 				)
@@
 		(on_board yes)
 		(dnp no)
-		(property "Reference" "Ra1"
+		(property "Reference" "Rw1"
 			(at 182.88 48.26 90)
 			(effects
@@
 			(project "gb-cart-arduino-v2"
 				(path "/9cf3a41e-ce13-4647-b5c2-ee25df0afcb2"
-					(reference "Ra1")
+					(reference "Rw1")
 					(unit 1)
 				)
@@
 		(on_board yes)
 		(dnp no)
-		(property "Reference" "Rd6"
+		(property "Reference" "Rd2"
 			(at 199.39 152.4 0)
 			(effects
@@
 			(project "gb-cart-arduino-v2"
 				(path "/9cf3a41e-ce13-4647-b5c2-ee25df0afcb2"
-					(reference "Rd6")
+					(reference "Rd2")
 					(unit 1)
 				)
@@
 		(on_board yes)
 		(dnp no)
-		(property "Reference" "Rd1"
+		(property "Reference" "Rd7"
 			(at 181.61 152.4 0)
 			(effects
@@
 			(project "gb-cart-arduino-v2"
 				(path "/9cf3a41e-ce13-4647-b5c2-ee25df0afcb2"
-					(reference "Rd1")
+					(reference "Rd7")
 					(unit 1)
 				)
@@
 		(on_board yes)
 		(dnp no)
-		(property "Reference" "Ra4"
+		(property "Reference" "Rl1"
 			(at 193.04 24.13 90)
 			(effects
@@
 			(project "gb-cart-arduino-v2"
 				(path "/9cf3a41e-ce13-4647-b5c2-ee25df0afcb2"
-					(reference "Ra4")
+					(reference "Rl1")
 					(unit 1)
 				)
@@
 		(on_board yes)
 		(dnp no)
-		(property "Reference" "Rd7"
+		(property "Reference" "Rd1"
 			(at 201.93 152.4 0)
 			(effects
@@
 			(project "gb-cart-arduino-v2"
 				(path "/9cf3a41e-ce13-4647-b5c2-ee25df0afcb2"
-					(reference "Rd7")
+					(reference "Rd1")
 					(unit 1)
 				)

Commit message: Reversed gb cart connector footprint
Parts:
- renumbered Rw1 to Rr1, Rr1 to Rw1
Connections:
- net Address_Clock: now also J1.6 (Pin_6); no longer J1.8 (Pin_8)
- net Address_Data: now also J1.8 (Pin_8); no longer J1.6 (Pin_6)
Changed lines of the file:
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@@
 	(wire
 		(pts
+			(xy 71.12 92.71) (xy 36.83 92.71)
+		)
+		(stroke
+			(width 0)
+			(type default)
+		)
+	)
+	(wire
+		(pts
 			(xy 50.8 82.55) (xy 36.83 82.55)
 		)
@@
 	(wire
 		(pts
+			(xy 76.2 64.77) (xy 76.2 97.79)
+		)
+		(stroke
+			(width 0)
+			(type default)
+		)
+	)
+	(wire
+		(pts
 			(xy 128.27 92.71) (xy 218.44 92.71)
 		)
@@
 	(wire
 		(pts
-			(xy 76.2 92.71) (xy 36.83 92.71)
-		)
-		(stroke
-			(width 0)
-			(type default)
-		)
-	)
-	(wire
-		(pts
 			(xy 90.17 123.19) (xy 102.87 123.19)
 		)
@@
 	(wire
 		(pts
-			(xy 80.01 69.85) (xy 80.01 97.79)
-		)
-		(stroke
-			(width 0)
-			(type default)
-		)
-	)
-	(wire
-		(pts
 			(xy 83.82 59.69) (xy 113.03 59.69)
 		)
@@
 	(wire
 		(pts
+			(xy 71.12 69.85) (xy 71.12 92.71)
+		)
+		(stroke
+			(width 0)
+			(type default)
+		)
+	)
+	(wire
+		(pts
 			(xy 177.8 45.72) (xy 177.8 58.42)
 		)
@@
 	(wire
 		(pts
+			(xy 36.83 97.79) (xy 76.2 97.79)
+		)
+		(stroke
+			(width 0)
+			(type default)
+		)
+	)
+	(wire
+		(pts
 			(xy 71.12 156.21) (xy 71.12 118.11)
 		)
@@
 	(wire
 		(pts
-			(xy 76.2 64.77) (xy 76.2 92.71)
-		)
-		(stroke
-			(width 0)
-			(type default)
-		)
-	)
-	(wire
-		(pts
 			(xy 215.9 158.75) (xy 215.9 143.51)
 		)
@@
 	(wire
 		(pts
-			(xy 80.01 69.85) (xy 96.52 69.85)
+			(xy 102.87 115.57) (xy 83.82 115.57)
 		)
 		(stroke
@@
 	(wire
 		(pts
-			(xy 102.87 115.57) (xy 83.82 115.57)
+			(xy 73.66 36.83) (xy 73.66 87.63)
 		)
 		(stroke
@@
 	(wire
 		(pts
-			(xy 73.66 36.83) (xy 73.66 87.63)
+			(xy 123.19 110.49) (xy 146.05 110.49)
 		)
 		(stroke
@@
 	(wire
 		(pts
-			(xy 123.19 110.49) (xy 146.05 110.49)
+			(xy 123.19 123.19) (xy 158.75 123.19)
 		)
 		(stroke
@@
 	(wire
 		(pts
-			(xy 123.19 123.19) (xy 158.75 123.19)
+			(xy 71.12 69.85) (xy 96.52 69.85)
 		)
 		(stroke
@@
 	(wire
 		(pts
-			(xy 36.83 97.79) (xy 80.01 97.79)
-		)
-		(stroke
-			(width 0)
-			(type default)
-		)
-	)
-	(wire
-		(pts
 			(xy 80.01 100.33) (xy 36.83 100.33)
 		)
@@
 	)
 	(label "Address_Clock"
-		(at 39.37 97.79 0)
+		(at 39.37 92.71 0)
 		(effects
 			(font
@@
 	)
 	(label "Address_Data"
-		(at 39.37 92.71 0)
+		(at 39.37 97.79 0)
 		(effects
 			(font
@@
 		(on_board yes)
 		(dnp no)
-		(property "Reference" "Rr1"
+		(property "Reference" "Rw1"
 			(at 182.88 52.07 90)
 			(effects
@@
 			(project "gb-cart-arduino-v2"
 				(path "/9cf3a41e-ce13-4647-b5c2-ee25df0afcb2"
-					(reference "Rr1")
+					(reference "Rw1")
 					(unit 1)
 				)
@@
 		(on_board yes)
 		(dnp no)
-		(property "Reference" "Rw1"
+		(property "Reference" "Rr1"
 			(at 182.88 48.26 90)
 			(effects
@@
 			(project "gb-cart-arduino-v2"
 				(path "/9cf3a41e-ce13-4647-b5c2-ee25df0afcb2"
-					(reference "Rw1")
+					(reference "Rr1")
 					(unit 1)
 				)

Commit message: Moved connector definition to project
Parts:
- U3: footprint 1_my_custom_library:Gameboy cartridge connector -> gb-cart:Gameboy cartridge connector; symbol 1_my_custom_library:GB_cartridge_connector -> gb-cart:GB_cartridge_connector
Changed lines of the file:
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@@
 	)
 	(symbol
-		(lib_id "1_my_custom_library:GB_cartridge_connector")
+		(lib_id "gb-cart:GB_cartridge_connector")
 		(at 233.68 104.14 0)
 		(unit 1)
@@
 			)
 		)
-		(property "Footprint" "1_my_custom_library:Gameboy cartridge connector"
+		(property "Footprint" "gb-cart:Gameboy cartridge connector"
 			(at 233.68 104.14 0)
 			(effects
